File: PCB/jazzette.kicad_pcb (KiCad board)
At the start: 2 copper layers, 95.6 x 54.4 mm, 25 parts, among them J1 Conn_02x08_Odd_Even, M1 Motor_DC, SW1 SMD_6.2x6.2mm_h7.0mm, SW2 SMD_6.2x6.2mm_h7.0mm, SW3 SMD_6.2x6.2mm_h7.0mm, SW5 SMD_6.2x6.2mm_h7.0mm, U2 DRV8833 breakout, U3 ESP32_S3_NANO

Commit message: board sent to mfg
Parts:
- removed R2: 1k, PCM_SparkFun-Resistor:R_0603_1608Metric
- added J2: Conn_01x02_Pin, EasyEDA_Lib:CONN-TH_DB125-2.54-2P-GN, F.Cu at (192.6, 106.1)
- added SW4: SW_Push_DPDT, Connector_PinHeader_2.54mm:PinHeader_1x04_P2.54mm_Vertical, F.Cu at (194.3, 119.4)
- added kobee-studio-6A9C82AE: Kobee Studio, kobee-studio-6A9C8293, B.Cu at (161.0, 96.0)
- added kobee-studio-6A9E54C5: Kobee Studio, kobee-studio-6A9E54C5, F.Cu at (150.7, 94.3)
- added kobee-studio-6A9E54DB: Kobee Studio, kobee-studio-6A9E54DB, F.Cu at (138.6, 94.3)
- added kobee-studio-6A9E5502: Kobee Studio, kobee-studio-6A9E54DB, F.Cu at (162.6, 94.3)
- added kobee-studio-6A9E550D: Kobee Studio, kobee-studio-6A9E54DB, F.Cu at (172.3, 94.3)
- added kobee-studio-6A9E5517: Kobee Studio, kobee-studio-6A9E54DB, F.Cu at (187.8, 94.5)
- added kobee-studio-6A9E55B7: Kobee Studio, kobee-studio-6A9E54DB, F.Cu at (145.4, 110.7)
- added kobee-studio-6A9E5BD7: Kobee Studio, kobee-studio-6A9E5478, F.Cu at (122.6, 89.5)
- added kobee-studio-6A9E5E3B: Kobee Studio, kobee-studio-6A9E5C65, B.Cu at (192.6, 104.8)
- added kobee-studio-6A9F86BB: Kobee Studio, kobee-studio-6A9F86BB, F.Cu at (191.4, 115.3)
- added kobee-studio-6A9F8757: Kobee Studio, kobee-studio-6A9F8711, B.Cu at (194.3, 111.8)
- SW1, SW2, SW3, SW5: footprint EasyEDA_Lib:SW-SMD_SH-6X6X4.5H-TP -> Circuits:SW-SMD_SH-6X6X4.5H-TP
- moved R1 6.95 mm to (147.4, 98.6), turned to 180 degrees
- moved C3 2.23 mm to (178.7, 94.2), turned to 180 degrees
- moved REF** 2.16 mm to (193.2, 99.4)
- moved SW2 0.08 mm to (145.9, 128.0)
- moved SW3 0.05 mm to (166.0, 128.0)
- renumbered kobee-studio-6A97BAF5 to kobee-studio-6A9DE86C
Connections:
- U3 pad 12: HP_DIN -> unconnected-(U3-Pad12)
- U3 pad 13: HP_BCK -> Net-(SW4-B-Pad2)
- U3 pad 14: HP_WS -> Net-(SW4-B-Pad1)
- U3 pad 15: NFC_SDA -> unconnected-(U3-Pad15)
- U3 pad 17: unconnected-(U3-Pad17) -> NFC_SCL
- U3 pad 18: unconnected-(U3-Pad18) -> NFC_SDA
- U3 pad 21: unconnected-(U3-Pad21) -> COAX_DIN
- U3 pad 37: COAX_DIN -> HP_BCK
- U3 pad 38: unconnected-(U3-Pad38) -> HP_DIN
- U3 pad 40: unconnected-(U3-Pad40) -> TOSLINK_DIN
- U3 pad 41: NFC_SCL -> MTR_PINA
- U3 pad 42: MTR_PINA -> MTR_PINB
- U3 pad 45: MTR_PINB -> MTR_SLP
- U3 pad 46: MTR_SLP -> unconnected-(U3-Pad46)
- U3 pad 48: TOSLINK_DIN -> HP_WS
Routing:
- net Net-(SW4-B-Pad2): track 0.00 -> 42.2 mm
- net Net-(SW4-B-Pad1): track 0.00 -> 39.9 mm
- net 5V: track 33.0 -> 66.1 mm
- net TOSLINK_DIN: track 24.6 -> 33.3 mm
- net BTN_D: track 40.7 -> 48.6 mm
- net BTN_A: track 19.0 -> 26.8 mm
- net BTN_C: track 22.4 -> 30.2 mm
- net BTN_B: track 6.02 -> 13.8 mm
- net HP_WS: track 51.0 -> 44.4 mm
- net NFC_SDA: track 29.8 -> 23.3 mm
- net HP_DIN: track 51.0 -> 44.8 mm
- net HP_BCK: track 50.4 -> 44.3 mm
- net Net-(CoaxJ2-In): track 14.3 -> 20.0 mm
- net NFC_SCL: track 30.2 -> 24.5 mm
- net +3V3: track 161.3 -> 163.8 mm, vias 1 -> 3
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