File: PCB/jazzette.kicad_sch (KiCad schematic)
At the start: 18 parts, among them J1 Conn_02x08_Odd_Even, M1 Motor_DC, SW1 SMD_6.2x6.2mm_h7.0mm, SW2 SMD_6.2x6.2mm_h7.0mm, SW3 SMD_6.2x6.2mm_h7.0mm, SW4 SW_SP3T, SW5 SMD_6.2x6.2mm_h7.0mm, U2 DRV8833 breakout, U3 ESP32_S3_NANO

Commit message: board sent to mfg
Parts:
- removed R2: 1k, PCM_SparkFun-Resistor:R_0603_1608Metric, symbol PCM_SparkFun-Resistor:R
- removed SW4: SW_SP3T, symbol Switch:SW_SP3T
- added J2: Conn_01x02_Pin, EasyEDA_Lib:CONN-TH_DB125-2.54-2P-GN, symbol Connector:Conn_01x02_Pin
- added SW4: SW_Push_DPDT, Connector_PinHeader_2.54mm:PinHeader_1x04_P2.54mm_Vertical, symbol Switch:SW_Push_DPDT
- SW1, SW2, SW3, SW5: footprint EasyEDA_Lib:SW-SMD_SH-6X6X4.5H-TP -> Circuits:SW-SMD_SH-6X6X4.5H-TP
Connections:
- net 5V: now also J2.1 (Pin_1)
- net COAX_DIN: now also U3.21; no longer U3.37
- net GND: now also J2.2 (Pin_2), SW4.3 (A), SW4.4 (A)
- net HP_BCK: now also U3.37; no longer U3.13
- net HP_DIN: now also U3.38; no longer U3.12
- net HP_WS: now also U3.48; no longer U3.14
- net MTR_PINA: now also U3.41; no longer U3.42
- net MTR_PINB: now also U3.42; no longer U3.45
- net MTR_SLP: now also U3.45; no longer U3.46
- net NFC_SCL: now also U3.17; no longer U3.41
- net NFC_SDA: now also U3.18; no longer U3.15
- net TOSLINK_DIN: now also U3.40; no longer U3.48
- new net: SW4.1 (B), U3.14
- new net: SW4.2 (B), U3.13
- no-connect marks 10 -> 22
